File: I2C-Oled-Backpack-Newhaven.brd (EAGLE design)
At the start: 50.8 x 19.1 mm, 17 parts, among them J1 4P-SMD-2.0-90D, J2 4P-SMD-2.0-90D, J3 LCD-NEWHAVEN-LOCK

Commit message: Rev B design
Parts:
- removed R5: 10K, 0:0805-RES
- removed SJ4: SOLDERJUMPERNC, 0:SJ_2S
Connections:
- removed net REGVDD: J3.3, R5.2, SJ4.2
- net GND: now also J3.3; no longer SJ4.1
- net VCC: no longer R5.1
Routing:
- net REGVDD: track 28.2 -> 0.00 mm
- net GND: track 16.5 -> 21.4 mm, vias 5 -> 4
Other:
- board text added: "(Rev B)"
- board text added: "I2C OLED BACKPACK - NEWHAVEN (Rev B)"
- board text removed: "(Rev A)"
- board text removed: "CLSD=3V"
- board text removed: "I2C OLED BACKPACK - NEWHAVEN (Rev A)"
- board text removed: "OPEN=5V"
- board text removed: "SELECT"
- board text removed: "VOLTS !!"
Changed lines of the file:
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@@
 <layers>
 <layer number="1" name="Top" color="4" fill="1" visible="yes" active="yes"/>
-<layer number="16" name="Bottom" color="1" fill="1" visible="yes" active="yes"/>
+<layer number="16" name="Bottom" color="1" fill="1" visible="no" active="yes"/>
 <layer number="17" name="Pads" color="2" fill="1" visible="yes" active="yes"/>
 <layer number="18" name="Vias" color="2" fill="1" visible="yes" active="yes"/>
@@
 <text x="32.2326" y="17.3228" size="0.889" layer="21" font="vector" ratio="11">I2C OLED BKPK NEWHAVEN</text>
 <text x="23.8506" y="18.1356" size="0.889" layer="21" font="vector" ratio="11">+</text>
-<text x="49.53" y="17.145" size="0.889" layer="22" font="vector" ratio="11" rot="MR0">I2C OLED BACKPACK - NEWHAVEN (Rev A)</text>
+<text x="49.53" y="17.145" size="0.889" layer="22" font="vector" ratio="11" rot="MR0">I2C OLED BACKPACK - NEWHAVEN (Rev B)</text>
 <text x="32.258" y="3.048" size="0.889" layer="21" font="vector" ratio="11" rot="R90">SDA</text>
 <text x="34.671" y="3.048" size="0.889" layer="21" font="vector" ratio="11" rot="R90">SCL</text>
@@
 <rectangle x1="10.4648" y1="14.4018" x2="12.5984" y2="15.8496" layer="43"/>
 <text x="7.747" y="16.891" size="1.524" layer="22" font="vector" ratio="10" rot="MR0">wht.io</text>
-<rectangle x1="28.2956" y1="13.8176" x2="29.972" y2="15.0114" layer="43"/>
-<text x="31.623" y="12.446" size="0.889" layer="21" font="vector" ratio="11" rot="R180">SELECT</text>
-<text x="32.512" y="13.462" size="0.889" layer="21" font="vector" ratio="11" rot="R180">VOLTS !!</text>
-<text x="32.258" y="7.493" size="0.889" layer="21" font="vector" ratio="11" rot="R180">OPEN=5V</text>
-<text x="32.258" y="8.636" size="0.889" layer="21" font="vector" ratio="11" rot="R180">CLSD=3V</text>
 <text x="18.288" y="7.62" size="0.889" layer="21" font="vector" ratio="11" rot="R180">C=3C</text>
 <text x="18.288" y="6.604" size="0.889" layer="21" font="vector" ratio="11" rot="R180">O=3D</text>
@@
 <rectangle x1="14.986" y1="5.588" x2="18.288" y2="8.763" layer="43"/>
 <rectangle x1="19.304" y1="4.699" x2="25.019" y2="5.969" layer="43"/>
-<rectangle x1="26.416" y1="6.604" x2="32.258" y2="9.017" layer="43"/>
-<rectangle x1="26.543" y1="11.43" x2="31.496" y2="13.589" layer="43"/>
-<text x="33.5026" y="16.0528" size="0.889" layer="21" font="vector" ratio="11">(Rev A)</text>
+<text x="33.5026" y="16.0528" size="0.889" layer="21" font="vector" ratio="11">(Rev B)</text>
 <rectangle x1="36.2966" y1="3.5306" x2="37.973" y2="4.7244" layer="43"/>
 <rectangle x1="38.9636" y1="3.4036" x2="40.64" y2="4.5974" layer="43"/>
@@
 <rectangle x1="26.035" y1="2.921" x2="29.337" y2="6.096" layer="43"/>
 <rectangle x1="16.8656" y1="2.7686" x2="18.542" y2="3.9624" layer="43"/>
-<rectangle x1="30.7975" y1="8.7757" x2="32.0167" y2="11.4427" layer="43" rot="R90"/>
 </plain>
 <attributes>
@@
 <attribute name="NAME" x="18.4912" y="3.7592" size="0.889" layer="25" font="vector" ratio="11" rot="R180"/>
 </element>
-<element name="SJ4" library="0" package="SJ_2S" value="SOLDERJUMPERNC" x="29.21" y="10.16" smashed="yes" rot="R90">
-<attribute name="NAME" x="32.6998" y="10.541" size="0.889" layer="25" rot="R180"/>
-</element>
-<element name="R5" library="0" package="0805-RES" value="10K" x="29.21" y="16.51" smashed="yes" rot="R270">
-<attribute name="NAME" x="30.099" y="14.7955" size="0.889" layer="25" font="vector" ratio="11" rot="R180"/>
-</element>
 <element name="J4" library="0" package="1X04_LOCK" value="" x="36.83" y="13.97" smashed="yes" rot="R270">
 <attribute name="NAME" x="38.0492" y="4.5212" size="0.889" layer="25" font="vector" ratio="11" rot="R180"/>
@@
 <contactref element="SJ3" pad="1"/>
 <contactref element="J3" pad="20"/>
-<contactref element="SJ4" pad="1"/>
 <contactref element="J3" pad="1"/>
 <contactref element="J3" pad="5"/>
@@
 <via x="18.161" y="9.652" extent="1-16" drill="0.508"/>
 <via x="25.527" y="14.351" extent="1-16" drill="0.508"/>
-<via x="27.559" y="9.652" extent="1-16" drill="0.508"/>
 <via x="42.926" y="7.112" extent="1-16" drill="0.508"/>
 <wire x1="40.54" y1="7.16" x2="42.926" y2="7.16" width="0.4064" layer="1"/>
@@
 <wire x1="37.846" y1="6.35" x2="38.608" y2="7.112" width="0.4064" layer="1"/>
 <wire x1="38.608" y1="7.112" x2="40.767" y2="7.112" width="0.4064" layer="1"/>
-<wire x1="29.21" y1="9.71" x2="27.617" y2="9.71" width="0.4064" layer="1"/>
-<wire x1="27.617" y1="9.71" x2="27.559" y2="9.652" width="0.4064" layer="1"/>
 <wire x1="16.51" y1="9.71" x2="18.103" y2="9.71" width="0.4064" layer="1"/>
 <wire x1="18.103" y1="9.71" x2="18.161" y2="9.652" width="0.4064" layer="1"/>
@@
 <wire x1="26.173" y1="15.113" x2="26.67" y2="15.61" width="0.4064" layer="1"/>
 <wire x1="25.527" y1="14.351" x2="25.527" y2="15.113" width="0.4064" layer="1"/>
+<contactref element="J3" pad="3"/>
+<wire x1="44.45" y1="1.143" x2="44.45" y2="2.54" width="0.1778" layer="1"/>
+<wire x1="44.45" y1="2.54" x2="43.18" y2="3.81" width="0.1778" layer="1"/>
+<wire x1="43.18" y1="3.81" x2="43.18" y2="6.858" width="0.1778" layer="1"/>
+<wire x1="43.18" y1="6.858" x2="42.926" y2="7.112" width="0.1778" layer="1"/>
 </signal>
 <signal name="SA0">
@@
 <contactref element="R4" pad="1"/>
 <contactref element="J3" pad="18"/>
-<contactref element="R5" pad="1"/>
 <contactref element="J3" pad="2"/>
 <contactref element="J4" pad="3"/>
@@
 <wire x1="24.13" y1="17.41" x2="24.13" y2="17.78" width="0.4064" layer="1"/>
 <wire x1="26.67" y1="17.41" x2="26.67" y2="17.78" width="0.4064" layer="1"/>
-<wire x1="29.21" y1="17.41" x2="29.21" y2="17.78" width="0.4064" layer="1"/>
 <wire x1="40.54" y1="9.16" x2="44.212" y2="9.16" width="0.4064" layer="1"/>
 <wire x1="44.212" y1="9.16" x2="44.45" y2="9.398" width="0.4064" layer="1"/>
@@
 <wire x1="20.2692" y1="10.668" x2="20.32" y2="10.61" width="0.1778" layer="1"/>
 </signal>
-<signal name="REGVDD">
-<contactref element="J3" pad="3"/>
-<contactref element="SJ4" pad="2"/>
-<contactref element="R5" pad="2"/>
-<wire x1="29.1592" y1="10.668" x2="29.1592" y2="15.4686" width="0.1778" layer="1"/>
-<wire x1="29.1592" y1="15.4686" x2="29.21" y2="15.61" width="0.1778" layer="1"/>
-<wire x1="29.1592" y1="10.668" x2="29.21" y2="10.61" width="0.1778" layer="1"/>
-<wire x1="44.45" y1="1.2446" x2="42.3164" y2="3.3782" width="0.1778" layer="1"/>
-<wire x1="29.337" y1="10.4902" x2="29.21" y2="10.61" width="0.1778" layer="1"/>
-<wire x1="44.45" y1="1.2446" x2="44.45" y2="1.143" width="0.1778" layer="1"/>
-<wire x1="42.3164" y1="3.3782" x2="30.9118" y2="3.3782" width="0.1778" layer="1"/>
-<wire x1="30.9118" y1="3.3782" x2="30.48" y2="3.81" width="0.1778" layer="1"/>
-<wire x1="30.48" y1="3.81" x2="30.48" y2="10.287" width="0.1778" layer="1"/>
-<wire x1="29.21" y1="10.61" x2="30.157" y2="10.61" width="0.1778" layer="1"/>
-<wire x1="30.157" y1="10.61" x2="30.48" y2="10.287" width="0.1778" layer="1"/>
-</signal>
 </signals>

Commit message: Rev C
Other:
- board text added: "(Rev C)"
- board text added: "I2C OLED BACKPACK - NEWHAVEN (Rev C)"
- board text added: "dcity.org"
- board text removed: "(Rev B)"
- board text removed: "I2C OLED BACKPACK - NEWHAVEN (Rev B)"
- board text removed: "wht.io"
Changed lines of the file:
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@@
 <?xml version="1.0" encoding="utf-8"?>
 <!DOCTYPE eagle SYSTEM "eagle.dtd">
-<eagle version="7.5.0">
+<eagle version="9.1.3">
 <drawing>
 <settings>
 <setting alwaysvectorfont="no"/>
+<setting keepoldvectorfont="yes"/>
 <setting verticaltext="up"/>
 </settings>
@@
 <layers>
 <layer number="1" name="Top" color="4" fill="1" visible="yes" active="yes"/>
-<layer number="16" name="Bottom" color="1" fill="1" visible="no" active="yes"/>
+<layer number="16" name="Bottom" color="1" fill="1" visible="yes" active="yes"/>
 <layer number="17" name="Pads" color="2" fill="1" visible="yes" active="yes"/>
 <layer number="18" name="Vias" color="2" fill="1" visible="yes" active="yes"/>
@@
 <text x="32.2326" y="17.3228" size="0.889" layer="21" font="vector" ratio="11">I2C OLED BKPK NEWHAVEN</text>
 <text x="23.8506" y="18.1356" size="0.889" layer="21" font="vector" ratio="11">+</text>
-<text x="49.53" y="17.145" size="0.889" layer="22" font="vector" ratio="11" rot="MR0">I2C OLED BACKPACK - NEWHAVEN (Rev B)</text>
+<text x="49.53" y="17.145" size="0.889" layer="22" font="vector" ratio="11" rot="MR0">I2C OLED BACKPACK - NEWHAVEN (Rev C)</text>
 <text x="32.258" y="3.048" size="0.889" layer="21" font="vector" ratio="11" rot="R90">SDA</text>
 <text x="34.671" y="3.048" size="0.889" layer="21" font="vector" ratio="11" rot="R90">SCL</text>
 <text x="49.784" y="2.921" size="0.889" layer="21" font="vector" ratio="11" rot="R90">G</text>
 <text x="47.371" y="2.921" size="0.889" layer="21" font="vector" ratio="11" rot="R90">V</text>
-<text x="1.524" y="16.9418" size="1.524" layer="21" font="vector" ratio="10">wht.io</text>
+<text x="1.524" y="16.9418" size="1.524" layer="21" font="vector" ratio="10">dcity.org</text>
 <rectangle x1="13.0556" y1="13.8176" x2="14.732" y2="15.0114" layer="43"/>
 <rectangle x1="15.621" y1="13.7922" x2="17.2212" y2="15.0622" layer="43"/>
@@
 <rectangle x1="48.8188" y1="2.54" x2="50.1904" y2="3.8608" layer="43"/>
 <rectangle x1="10.4648" y1="14.4018" x2="12.5984" y2="15.8496" layer="43"/>
-<text x="7.747" y="16.891" size="1.524" layer="22" font="vector" ratio="10" rot="MR0">wht.io</text>
+<text x="11.557" y="16.891" size="1.524" layer="22" font="vector" ratio="10" rot="MR0">dcity.org</text>
 <text x="18.288" y="7.62" size="0.889" layer="21" font="vector" ratio="11" rot="R180">C=3C</text>
 <text x="18.288" y="6.604" size="0.889" layer="21" font="vector" ratio="11" rot="R180">O=3D</text>
@@
 <rectangle x1="14.986" y1="5.588" x2="18.288" y2="8.763" layer="43"/>
 <rectangle x1="19.304" y1="4.699" x2="25.019" y2="5.969" layer="43"/>
-<text x="33.5026" y="16.0528" size="0.889" layer="21" font="vector" ratio="11">(Rev B)</text>
+<text x="33.5026" y="16.0528" size="0.889" layer="21" font="vector" ratio="11">(Rev C)</text>
 <rectangle x1="36.2966" y1="3.5306" x2="37.973" y2="4.7244" layer="43"/>
 <rectangle x1="38.9636" y1="3.4036" x2="40.64" y2="4.5974" layer="43"/>
@@
 <rectangle x1="26.035" y1="2.921" x2="29.337" y2="6.096" layer="43"/>
 <rectangle x1="16.8656" y1="2.7686" x2="18.542" y2="3.9624" layer="43"/>
+<wire x1="50.8" y1="19.05" x2="50.8" y2="0" width="0" layer="20"/>
 </plain>
 <attributes>
@@
 <param name="dpMaxLengthDifference" value="10mm"/>
 <param name="dpGapFactor" value="2.5"/>
-<param name="checkGrid" value="0"/>
 <param name="checkAngle" value="1"/>
 <param name="checkFont" value="1"/>
 <param name="checkRestrict" value="1"/>
+<param name="checkStop" value="0"/>
+<param name="checkValues" value="0"/>
+<param name="checkNames" value="1"/>
+<param name="checkWireStubs" value="1"/>
+<param name="checkPolygonWidth" value="0"/>
 <param name="useDiameter" value="13"/>
 <param name="maxErrors" value="50"/>
@@
 </signal>
 </signals>
+<mfgpreviewcolors>
+<mfgpreviewcolor name="soldermaskcolor" color="0xC8008000"/>
+<mfgpreviewcolor name="silkscreencolor" color="0xFFFEFEFE"/>
+<mfgpreviewcolor name="backgroundcolor" color="0xFF282828"/>
+<mfgpreviewcolor name="coppercolor" color="0xFFFFBF00"/>
+<mfgpreviewcolor name="substratecolor" color="0xFF786E46"/>
+</mfgpreviewcolors>
 </board>
 </drawing>

Commit message: Rev D
Parts:
- J1, J2: value 4P-SMD-2.0-90D -> QWIIC_RIGHT_ANGLE; device 0:HW4-SMD-2.0-90D -> 0:JST04_1MM_RA
- moved J2 5.12 mm to (5.08, 9.53), turned to 270 degrees
- moved J1 4.99 mm to (45.6, 9.53), turned to 90 degrees
Connections:
- net GND: now also J1.1, J2.1; no longer J1.4, J2.4
- net SCL: now also J1.4, J2.4; no longer J1.1, J2.1
- net SDA: now also J1.3, J2.3; no longer J1.2, J2.2
- net VCC: now also J1.2, J2.2; no longer J1.3, J2.3
Routing:
- net SDA: track 65.6 -> 81.4 mm
- net GND: track 21.4 -> 11.2 mm
- net SCL: track 65.5 -> 72.0 mm
- net VCC: track 82.9 -> 85.4 mm
Other:
- board text added: "(Rev D)"
- board text added: "GND"
- board text added: "I2C OLED BACKPACK - NEWHAVEN (Rev D)"
- board text added: "VCC"
- board text removed: "(Rev C)"
- board text removed: "I2C OLED BACKPACK - NEWHAVEN (Rev C)"
