File: I2C-Oled-Backpack-Newhaven.sch (EAGLE design)
At the start: 17 parts, among them J1 4P-SMD-2.0-90D, J2 4P-SMD-2.0-90D, J3 LCD-NEWHAVEN-LOCK

Commit message: Rev B design
Parts:
- removed R5: 10K, 0:RESISTOR0805
- removed SJ4: SOLDERJUMPERNC, 0:SOLDERJUMPERNC
Connections:
- removed net REGVDD: J3.REGVDD, R5.2, SJ4.2
- net GND: now also J3.REGVDD; no longer SJ4.1
- net VCC: no longer R5.1
Other:
- note removed: "CLOSED=3.3V"
- note removed: "IMPORTANT !!! SET JUMPER BEFORE USE !!!"
- note removed: "OPEN=5V"
- note removed: "Voltage Select"
Changed lines of the file:
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@@
 <setting verticaltext="up"/>
 </settings>
-<grid distance="0.1" unitdist="inch" unit="inch" style="lines" multiple="1" display="yes" altdistance="0.05" altunitdist="inch" altunit="inch"/>
+<grid distance="0.1" unitdist="inch" unit="inch" style="lines" multiple="1" display="no" altdistance="0.01" altunitdist="inch" altunit="inch"/>
 <layers>
 <layer number="1" name="Top" color="4" fill="1" visible="no" active="no"/>
@@
 <attribute name="DRAWNBY" value="Gary Muhonen"/>
 <attribute name="TITLE" value="I2C OLED Backpack (Newhaven)"/>
-<attribute name="VERSION" value="A"/>
+<attribute name="VERSION" value="B"/>
 </part>
 <part name="C1" library="0" deviceset="CAP" device="0805" value="100NF"/>
@@
 <part name="U$2" library="0" deviceset="CREATIVE_COMMONS" device=""/>
 <part name="J3" library="0" deviceset="LCD-NEWHAVEN" device="-LOCK"/>
-<part name="SJ4" library="0" deviceset="SOLDERJUMPER" device="NC"/>
-<part name="R5" library="0" deviceset="RESISTOR" device="0805" value="10K"/>
-<part name="GND5" library="0 - Seeedstudio" deviceset="GND" device=""/>
-<part name="P+7" library="0 - Seeedstudio" deviceset="VCC" device=""/>
 <part name="GND8" library="0 - Seeedstudio" deviceset="GND" device=""/>
 <part name="J4" library="0" deviceset="M04" device="LOCK"/>
@@
 <text x="101.6" y="144.78" size="1.778" layer="91">jump=3C</text>
 <text x="73.66" y="154.94" size="1.778" layer="91">I2C Pullups</text>
-<text x="17.78" y="149.86" size="1.778" layer="91">Voltage Select</text>
-<text x="17.78" y="147.32" size="1.778" layer="91">OPEN=5V</text>
-<text x="17.78" y="144.78" size="1.778" layer="91">CLOSED=3.3V</text>
-<text x="15.24" y="134.62" size="1.778" layer="91">IMPORTANT !!!
-SET JUMPER
-BEFORE USE !!!</text>
 <text x="161.29" y="69.85" size="1.778" layer="91">OLED (Newhaven)</text>
 </plain>
@@
 <attribute name="NAME" x="160.02" y="127.508" size="1.778" layer="95"/>
 </instance>
-<instance part="SJ4" gate="1" x="43.18" y="149.86" rot="R90"/>
-<instance part="R5" gate="G$1" x="43.18" y="165.1" rot="R270"/>
-<instance part="GND5" gate="1" x="43.18" y="139.7"/>
-<instance part="P+7" gate="G$1" x="43.18" y="172.72"/>
 <instance part="GND8" gate="1" x="91.44" y="101.6"/>
 <instance part="J4" gate="G$1" x="78.74" y="116.84" rot="MR180"/>
@@
 <wire x1="147.32" y1="101.6" x2="147.32" y2="111.76" width="0.1524" layer="91"/>
 <wire x1="147.32" y1="111.76" x2="147.32" y2="114.3" width="0.1524" layer="91"/>
-<wire x1="147.32" y1="114.3" x2="147.32" y2="124.46" width="0.1524" layer="91"/>
+<wire x1="147.32" y1="114.3" x2="147.32" y2="119.38" width="0.1524" layer="91"/>
+<wire x1="147.32" y1="119.38" x2="147.32" y2="124.46" width="0.1524" layer="91"/>
 <wire x1="147.32" y1="124.46" x2="157.48" y2="124.46" width="0.1524" layer="91"/>
 <wire x1="157.48" y1="99.06" x2="147.32" y2="99.06" width="0.1524" layer="91"/>
@@
 <pinref part="J3" gate="G$1" pin="BS0"/>
 <pinref part="J3" gate="G$1" pin="BS2"/>
+<pinref part="J3" gate="G$1" pin="REGVDD"/>
+<wire x1="157.48" y1="119.38" x2="147.32" y2="119.38" width="0.1524" layer="91"/>
+<junction x="147.32" y="119.38"/>
 </segment>
 <segment>
@@
 <pinref part="SJ3" gate="1" pin="1"/>
 <wire x1="121.92" y1="142.24" x2="121.92" y2="144.78" width="0.1524" layer="91"/>
-</segment>
-<segment>
-<pinref part="GND5" gate="1" pin="GND"/>
-<pinref part="SJ4" gate="1" pin="1"/>
-<wire x1="43.18" y1="142.24" x2="43.18" y2="144.78" width="0.1524" layer="91"/>
 </segment>
 <segment>
@@
 </segment>
 <segment>
-<pinref part="R5" gate="G$1" pin="1"/>
-<pinref part="P+7" gate="G$1" pin="VCC"/>
-<wire x1="43.18" y1="170.18" x2="43.18" y2="172.72" width="0.1524" layer="91"/>
-</segment>
-<segment>
 <label x="86.36" y="114.3" size="1.778" layer="95" xref="yes"/>
 <pinref part="J4" gate="G$1" pin="3"/>
@@
 <pinref part="SJ2" gate="1" pin="2"/>
 <wire x1="91.44" y1="157.48" x2="91.44" y2="154.94" width="0.1524" layer="91"/>
-</segment>
-</net>
-<net name="REGVDD" class="0">
-<segment>
-<pinref part="J3" gate="G$1" pin="REGVDD"/>
-<wire x1="157.48" y1="119.38" x2="134.62" y2="119.38" width="0.1524" layer="91"/>
-<label x="134.62" y="119.38" size="1.778" layer="95" rot="R180" xref="yes"/>
-<label x="38.1" y="157.48" size="1.778" layer="95" rot="R180" xref="yes"/>
-</segment>
-<segment>
-<pinref part="SJ4" gate="1" pin="2"/>
-<pinref part="R5" gate="G$1" pin="2"/>
-<wire x1="43.18" y1="154.94" x2="43.18" y2="157.48" width="0.1524" layer="91"/>
-<wire x1="43.18" y1="157.48" x2="43.18" y2="160.02" width="0.1524" layer="91"/>
-<wire x1="38.1" y1="157.48" x2="43.18" y2="157.48" width="0.1524" layer="91"/>
-<junction x="43.18" y="157.48"/>
 </segment>
 </net>
@@
 </schematic>
 </drawing>
-<compatibility>
-<note version="6.3" minversion="6.2.2" severity="warning">
-Since Version 6.2.2 text objects can contain more than one line,
-which will not be processed correctly with this version.
-</note>
-</compatibility>
 </eagle>

Commit message: Rev D
Parts:
- J1, J2: value 4P-SMD-2.0-90D -> QWIIC_RIGHT_ANGLE; device 0:GROVE-CONNECTOR-SMD-90D(4+2P-2.0) -> 0:QWIIC_CONNECTORJS-1MM
Connections:
- net GND: now also J1.1, J2.1; no longer J1.4, J2.4
- net SCL: now also J1.4, J2.4; no longer J1.1, J2.1
- net SDA: now also J1.3, J2.3; no longer J1.2, J2.2
- net VCC: now also J1.2, J2.2; no longer J1.3, J2.3
